File: applebrd.kicad_pcb (KiCad board)
At the start: 2 copper layers, 355.6 x 215.9 mm, 155 parts, among them J1 Jack-DC, J10 Conn_02x25_Counter_Clockwise_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, J11 Conn_02x25_Counter_Clockwise_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, J2 Jack-DC, J3 RCJ-014, J4 Conn_02x25_Counter_Clockwise_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, J5 Conn_02x25_Counter_Clockwise_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, J6 Conn_02x25_Counter_Clockwise_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, J7 Conn_02x25_Counter_Clockwise_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, J8 Conn_02x25_Counter_Clockwise_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, J9 Conn_02x25_Counter_Clockwise_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, Q2 2N3904, Q3 2N3904, Q4 Q_NPN_Darlington_EBC, Q5 2N3904, X1 CXO_DIP14

Commit message: Add files via upload
Ram chp wiring fixed.
Parts:
- added RN1: R_Network07_US, Resistor_THT:R_Array_SIP8, F.Cu at (210.8, 299.0)
- UE10, UE3, UE4, UE5, UE6, UE7, UE8, UE9: footprint Package_DIP:DIP-16_W7.62mm -> Package_DIP:DIP-18_W7.62mm
- moved JP1 53.7 mm to (159.8, 306.1)
- moved JP3 43.9 mm to (161.4, 358.5)
- moved UD2 0.50 mm to (172.6, 183.7)
- moved UE10 0.14 mm to (210.8, 296.0)
- turned R24 to 90 degrees
Connections:
- net /CAS renamed /~CAS
- net /MBL renamed /HBL
- net /NOMIX_MIX renamed /MIX_MODE
- net /RAS renamed /~RAS
- net /~COPS renamed /~LDPS
- net Net-(UB8-Pad6) renamed /RDO7
- J10 pad 19: (no net) -> Net-(J10-Pad19)
- J10 pad 35: (no net) -> Net-(J10-Pad35)
- J10 pad 38: /P1 -> /P0
- J11 pad 19: (no net) -> Net-(J11-Pad19)
- J11 pad 23: (no net) -> /INT_OUT
- J11 pad 24: (no net) -> /DMA_OUT
- J11 pad 29: (no net) -> Net-(J11-Pad29)
- J11 pad 30: (no net) -> Net-(J11-Pad30)
- J11 pad 31: (no net) -> Net-(J11-Pad31)
- J11 pad 32: (no net) -> Net-(J11-Pad32)
- J11 pad 33: (no net) -> Net-(J11-Pad33)
- J11 pad 34: (no net) -> Net-(J11-Pad34)
- J11 pad 35: (no net) -> Net-(J11-Pad35)
- J11 pad 38: /P1 -> /P0
- J4 pad 1: (no net) -> Net-(J4-Pad1)
- J4 pad 19: (no net) -> Net-(J4-Pad19)
- J4 pad 27: (no net) -> Net-(J4-Pad27)
- J4 pad 28: (no net) -> Net-(J4-Pad28)
- J4 pad 35: (no net) -> Net-(J4-Pad35)
- J4 pad 38: /P1 -> /P0
- J5 pad 19: (no net) -> Net-(J5-Pad19)
- J5 pad 35: (no net) -> Net-(J5-Pad35)
- J5 pad 38: /P1 -> /P0
- J6 pad 19: (no net) -> Net-(J6-Pad19)
- J6 pad 35: (no net) -> Net-(J6-Pad35)
- J6 pad 38: /P1 -> /P0
- J7 pad 19: (no net) -> Net-(J7-Pad19)
- J7 pad 35: (no net) -> Net-(J7-Pad35)
- J7 pad 38: /P1 -> /P0
- J8 pad 19: (no net) -> Net-(J8-Pad19)
- J8 pad 35: (no net) -> Net-(J8-Pad35)
- J8 pad 38: /P1 -> /P0
- J9 pad 19: (no net) -> Net-(J9-Pad19)
- J9 pad 35: (no net) -> Net-(J9-Pad35)
- J9 pad 38: /P1 -> /P0
- RN2 pad 2: (no net) -> Net-(RN2-Pad2)
- UA10 pad 10: /B12-8 -> /14M
- UA10 pad 12: (no net) -> Net-(UA10-Pad12)
- UA10 pad 6: (no net) -> Net-(UA10-Pad6)
- UA10 pad 7: (no net) -> Net-(UA10-Pad7)
- UA10 pad 9: /B12-8 -> /14M
- UA11 pad 12: (no net) -> Net-(UA11-Pad12)
- UA11 pad 5: (no net) -> Net-(UA11-Pad5)
- UA11 pad 7: (no net) -> Net-(UA11-Pad7)
- UA11 pad 8: (no net) -> Net-(UA11-Pad8)
- UA13 pad 5: (no net) -> Net-(UA13-Pad5)
- UA13 pad 7: (no net) -> Net-(UA13-Pad7)
- UA2 pad 1: /P1 -> /P0
- UA3 pad 1: Net-(UA3-Pad1) -> Net-(UA10-Pad12)
- UA3 pad 14: GND -> Net-(UA3-Pad14)
- UA3 pad 2: Net-(UA3-Pad2) -> Net-(UA10-Pad6)
- UA3 pad 3: GND -> Net-(UA3-Pad3)
- UA4 pad 10: Net-(UA3-Pad5) -> Net-(UA3-Pad14)
- UA4 pad 11: Net-(UA3-Pad10) -> Net-(UA3-Pad3)
- UA4 pad 13: Net-(UA3-Pad11) -> Net-(UA3-Pad12)
- UA4 pad 14: Net-(UA3-Pad12) -> Net-(UA3-Pad11)
- UA4 pad 15: (no net) -> Net-(UA3-Pad10)
- UA4 pad 16: (no net) -> Net-(UA3-Pad5)
- UA4 pad 17: (no net) -> Net-(UA3-Pad4)
- UA4 pad 20: (no net) -> GND
- UA4 pad 21: (no net) -> GND
- UA4 pad 22: (no net) -> GND
- UA4 pad 6: /VC -> /V0
- UA4 pad 7: /VB -> /V1
- UA4 pad 9: Net-(UA3-Pad4) -> Net-(UA4-Pad9)
- UA7 pad 15: (no net) -> Net-(UA7-Pad15)
- UA8 pad 11: (no net) -> Net-(UA8-Pad11)
- UA8 pad 3: /VC -> /V0
- UA8 pad 5: (no net) -> Net-(UA8-Pad5)
- UA8 pad 6: (no net) -> Net-(UA8-Pad6)
- UA9 pad 6: (no net) -> Net-(UA9-Pad6)
- UB1 pad 1: (no net) -> Net-(UB1-Pad1)
- UB1 pad 2: (no net) -> /~CREF
- UB1 pad 7: /P1 -> /P0
- UB10 pad 6: (no net) -> Net-(UB10-Pad6)
- UB10 pad 8: (no net) -> Net-(UB10-Pad8)
- UB11 pad 13: /D6 -> /RDL6
- UB12 pad 10: (no net) -> /P0
- UB12 pad 11: (no net) -> Net-(UA2-Pad2)
- UB12 pad 2: /H4 -> /H3
- UB12 pad 4: /V3 -> /V4
- UB12 pad 8: /B12-8 -> /14M
- UB12 pad 9: (no net) -> /7M
- UB13 pad 3: /H2 -> /H1
- UB13 pad 4: Net-(UA3-Pad2) -> Net-(UA10-Pad6)
- UB13 pad 6: /D7 -> /RDL7
- UB14 pad 8: /VC -> /V0
- UB2 pad 12: Net-(UA3-Pad1) -> Net-(UA10-Pad12)
- UB2 pad 2: Net-(UB1-Pad11) -> /~CREF
- UB2 pad 5: /H5 -> /~HPE
- UB3 pad 5: (no net) -> Net-(UB3-Pad5)
- UB4 pad 12: (no net) -> Net-(UB4-Pad12)
- UB4 pad 14: (no net) -> Net-(UB4-Pad14)
- UB4 pad 3: (no net) -> Net-(UB4-Pad3)
- UB4 pad 4: (no net) -> Net-(UB4-Pad4)
- UB4 pad 5: (no net) -> Net-(UB4-Pad5)
- UB4 pad 6: (no net) -> Net-(UB4-Pad6)
- UB4 pad 9: /B12-8 -> /14M
- UB5 pad 14: (no net) -> Net-(UB5-Pad14)
- UB5 pad 15: (no net) -> Net-(UB5-Pad15)
- UB9 pad 12: (no net) -> Net-(UB9-Pad12)
- UB9 pad 14: (no net) -> Net-(UB9-Pad14)
- UB9 pad 3: (no net) -> Net-(UB9-Pad3)
- UB9 pad 4: (no net) -> Net-(UB9-Pad4)
- UB9 pad 5: (no net) -> Net-(UB9-Pad5)
- UB9 pad 6: (no net) -> Net-(UB9-Pad6)
- UB9 pad 7: (no net) -> Net-(UB9-Pad7)
- UB9 pad 9: /B12-8 -> /14M
- UC12 pad 1: (no net) -> Net-(UC12-Pad1)
- UC12 pad 13: /VC -> /V0
- UC12 pad 4: (no net) -> Net-(UC12-Pad4)
- UC12 pad 6: /VB -> /V1
- UC12 pad 7: (no net) -> Net-(UC12-Pad7)
- UC13 pad 10: /H3 -> /H0
- UC13 pad 11: /H3 -> /H0
- UC2 pad 1: (no net) -> /SOFT-5
- UC2 pad 9: (no net) -> /Q3
- UC9 pad 3: (no net) -> Net-(UC9-Pad3)
- UD11 pad 11: /V2 -> /V5
- UD11 pad 12: /V3 -> /V4
- UD11 pad 13: /V4 -> /V3
- UD11 pad 14: /V5 -> /V2
- UD12 pad 11: /VB -> /V1
- UD12 pad 12: /VC -> /V0
- UD13 pad 11: /H4 -> /VA
- UD13 pad 12: /H5 -> /~HPE
- UD13 pad 13: (no net) -> /H5
- UD13 pad 14: /VA -> /H4
- UD13 pad 6: /H4 -> /VA
- UD13 pad 9: /H5 -> /~HPE
- UD14 pad 11: /H0 -> /H3
- UD14 pad 12: /H1 -> /H2
- UD14 pad 13: /H2 -> /H1
- UD14 pad 14: /H3 -> /H0
- UD14 pad 9: /H5 -> /~HPE
- UD2 pad 2: Net-(UB1-Pad11) -> /~CREF
- UD2 pad 5: /P1 -> /P0
- UD7 pad 14: (no net) -> /RDO4
- UD8 pad 14: (no net) -> /RDO5
- UE11 pad 10: (no net) -> Net-(UE11-Pad10)
- UE11 pad 6: (no net) -> Net-(UE11-Pad6)
- UE14 pad 14: /Y3 -> /V3
- UE14 pad 7: /Y3 -> /V3
- UE14 pad 9: (no net) -> Net-(UE14-Pad9)
- UE2 pad 1: (no net) -> Net-(UE2-Pad1)
- UE2 pad 6: (no net) -> Net-(UE2-Pad6)
- UE8 pad 15: (no net) -> Net-(UE8-Pad15)
- UE9 pad 15: (no net) -> Net-(UE9-Pad15)
- UF12 pad 4: /P1 -> /P0
- UF13 pad 12: /SPEAKER -> /SOFT-5
- UF14 pad 6: (no net) -> /PAGE1_PAGE2
- UF2 pad 7: (no net) -> Net-(UF2-Pad7)
- UF2 pad 9: (no net) -> Net-(UF2-Pad9)
- UG1 pad 13: /VC -> /V0
- UG1 pad 3: (no net) -> Net-(UG1-Pad3)
- UG1 pad 9: (no net) -> /PAGE2
- UG14 pad 6: (no net) -> Net-(UG14-Pad6)
- UG2 pad 5: /P1 -> /P0
- UH1 pad 2: (no net) -> Net-(UH1-Pad2)
- UH1 pad 4: (no net) -> Net-(UH1-Pad4)
- UH1 pad 7: (no net) -> Net-(UH1-Pad7)
- UH7 pad 35: (no net) -> Net-(UH7-Pad35)
- UH7 pad 36: (no net) -> Net-(UH7-Pad36)
- UH7 pad 39: (no net) -> Net-(UH7-Pad39)
- UH7 pad 5: (no net) -> Net-(UH7-Pad5)
- UH7 pad 7: (no net) -> Net-(UH7-Pad7)
- UH7 pad 8: (no net) -> Net-(UH7-Pad8)
- UJ13 pad 1: /SOFT-5 -> Net-(UJ13-Pad1)
- UJ13 pad 10: /SOFT-5 -> Net-(UJ13-Pad1)
- UJ13 pad 13: /SOFT-5 -> Net-(UJ13-Pad1)
- UJ13 pad 2: /SOFT-5 -> Net-(UJ13-Pad1)
- UJ13 pad 3: /SPEAKER -> /SOFT-5
- UJ13 pad 6: /SOFT-5 -> Net-(UJ13-Pad1)
- UJ13 pad 9: (no net) -> Net-(UJ13-Pad9)
- UK13 pad 1: (no net) -> Net-(UK13-Pad1)
- UK13 pad 5: (no net) -> Net-(UK13-Pad5)
- UK13 pad 8: (no net) -> Net-(UK13-Pad8)
- UM3 pad 13: (no net) -> Net-(UM3-Pad13)
- UM3 pad 14: (no net) -> Net-(UM3-Pad14)
Routing:
- net Net-(UA10-Pad5): track 0.00 -> 582.9 mm, vias 0 -> 2
- net /V0: track 0.00 -> 533.5 mm, vias 0 -> 8
- net /P0: track 203.2 -> 663.5 mm, vias 1 -> 10
- net /SOFT5_11: track 0.00 -> 379.0 mm, vias 0 -> 1
- net /HIRES: track 0.00 -> 333.3 mm, vias 0 -> 3
- net /H0: track 0.00 -> 264.6 mm, vias 0 -> 8
- net Net-(Q4-Pad3): track 0.00 -> 261.1 mm, vias 0 -> 2
- net /RD_KBD: track 0.00 -> 228.5 mm, vias 0 -> 3
- net (no net): track 1563.6 -> 1339.1 mm
- net Net-(UA2-Pad2): track 0.00 -> 204.7 mm, vias 0 -> 2
- net Net-(R5-Pad2): track 0.00 -> 193.7 mm, vias 0 -> 2
- net /A13: track 156.7 -> 348.7 mm, vias 1 -> 3
- net /MIX_MODE: track 0.00 -> 180.9 mm, vias 0 -> 2
- net /CREF: track 0.00 -> 180.6 mm
- net /A6: track 247.9 -> 426.3 mm, vias 0 -> 5
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- added copper zone on In1.Cu, net +5V
- added copper zone on In2.Cu, net GND
Other:
- copper layers 2 -> 4
